File: pcb/kicad/litvinov_oled_carrier.kicad_pcb (KiCad board)
At the start: 2 copper layers, 52 x 82 mm, 9 parts, among them J1 OLED 1x04: P1 P2 SCL SDA, J2 PASSIVE PIEZO, J3 18650 B+ B-, U1 ESP32-C3 SuperMini — measure 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

Commit message: fix: map ESP32-C3 SuperMini header pinout
Parts:
- U1: value ESP32-C3 SuperMini — measure before ordering -> ESP32-C3 SuperMini; USB end is at top; footprint Custom:ESP32-C3-SuperMini_SOCKET_TBC -> Custom:ESP32-C3-SuperMini_1x08_1x09
Changed lines of the file:
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@@
     (pad "GND" thru_hole circle (at 7 0) (size 2 2) (drill 1) (layers "*.Cu" "*.Mask") (net 2 "GND"))
   )
-  (footprint "Custom:ESP32-C3-SuperMini_SOCKET_TBC" (layer "F.Cu") (at 30 40)
-    (property "Reference" "U1" (at 10 0 0) (layer "F.SilkS") (effects (font (size 1.4 1.4) (thickness 0.25))))
-    (property "Value" "ESP32-C3 SuperMini — measure before ordering" (at 10 28 0) (layer "F.Fab") (effects (font (size 0.9 0.9) (thickness 0.14))))
-    (fp_rect (start -2 -2) (end 22 25) (stroke (width 0.4) (type dash)) (fill none) (layer "F.SilkS"))
-    (fp_text user "SUPERMINI SOCKET\nPIN SPACING TBC" (at 10 11) (layer "F.SilkS") (effects (font (size 1.2 1.2) (thickness 0.2)) (justify)))
-    (pad "GPIO4" thru_hole rect (at 0 0) (size 2 2) (drill 1) (layers "*.Cu" "*.Mask") (net 7 "BUZZER_PWM_GPIO4"))
-    (pad "GPIO8" thru_hole circle (at 0 2.54) (size 2 2) (drill 1) (layers "*.Cu" "*.Mask") (net 6 "I2C_SDA_GPIO8"))
-    (pad "GPIO9" thru_hole circle (at 0 5.08) (size 2 2) (drill 1) (layers "*.Cu" "*.Mask") (net 5 "I2C_SCL_GPIO9"))
-    (pad "GPIO3?" thru_hole circle (at 20 0) (size 2 2) (drill 1) (layers "*.Cu" "*.Mask") (net 9 "ADC_BAT_GPIO3"))
-    (pad "3V3" thru_hole circle (at 20 2.54) (size 2 2) (drill 1) (layers "*.Cu" "*.Mask") (net 1 "+3V3"))
-    (pad "GND" thru_hole circle (at 20 5.08) (size 2 2) (drill 1) (layers "*.Cu" "*.Mask") (net 2 "GND"))
+  (footprint "Custom:ESP32-C3-SuperMini_1x08_1x09" (layer "F.Cu") (at 30 40)
+    (property "Reference" "U1" (at 8.89 -3 0) (layer "F.SilkS") (effects (font (size 1.4 1.4) (thickness 0.25))))
+    (property "Value" "ESP32-C3 SuperMini; USB end is at top" (at 8.89 26 0) (layer "F.Fab") (effects (font (size 0.9 0.9) (thickness 0.14))))
+    (fp_rect (start -2 -2) (end 19.78 23) (stroke (width 0.4) (type dash)) (fill none) (layer "F.SilkS"))
+    (fp_text user "USB" (at 8.89 -0.3) (layer "F.SilkS") (effects (font (size 0.9 0.9) (thickness 0.14))))
+    (fp_text user "ESP32-C3\nSuperMini" (at 8.89 14) (layer "F.SilkS") (effects (font (size 1.1 1.1) (thickness 0.18)) (justify)))
+    (fp_text user "L: 5 6 7 8 9 10 20 21" (at -0.7 22.3) (layer "F.SilkS") (effects (font (size 0.65 0.65) (thickness 0.1)) (justify left)))
+    (fp_text user "R: 5V G 3V3 RST 4 3 2 1 0" (at 19.1 22.3) (layer "F.SilkS") (effects (font (size 0.65 0.65) (thickness 0.1)) (justify right)))
+    (pad "GPIO5" thru_hole rect (at 0 0) (size 2 2) (drill 1) (layers "*.Cu" "*.Mask"))
+    (pad "GPIO6" thru_hole circle (at 0 2.54) (size 2 2) (drill 1) (layers "*.Cu" "*.Mask"))
+    (pad "GPIO7" thru_hole circle (at 0 5.08) (size 2 2) (drill 1) (layers "*.Cu" "*.Mask"))
+    (pad "GPIO8" thru_hole circle (at 0 7.62) (size 2 2) (drill 1) (layers "*.Cu" "*.Mask") (net 6 "I2C_SDA_GPIO8"))
+    (pad "GPIO9" thru_hole circle (at 0 10.16) (size 2 2) (drill 1) (layers "*.Cu" "*.Mask") (net 5 "I2C_SCL_GPIO9"))
+    (pad "GPIO10" thru_hole circle (at 0 12.70) (size 2 2) (drill 1) (layers "*.Cu" "*.Mask"))
+    (pad "GPIO20" thru_hole circle (at 0 15.24) (size 2 2) (drill 1) (layers "*.Cu" "*.Mask"))
+    (pad "GPIO21" thru_hole circle (at 0 17.78) (size 2 2) (drill 1) (layers "*.Cu" "*.Mask"))
+    (pad "5V" thru_hole rect (at 17.78 0) (size 2 2) (drill 1) (layers "*.Cu" "*.Mask"))
+    (pad "GND" thru_hole circle (at 17.78 2.54) (size 2 2) (drill 1) (layers "*.Cu" "*.Mask") (net 2 "GND"))
+    (pad "3V3" thru_hole circle (at 17.78 5.08) (size 2 2) (drill 1) (layers "*.Cu" "*.Mask") (net 1 "+3V3"))
+    (pad "RST" thru_hole circle (at 17.78 7.62) (size 2 2) (drill 1) (layers "*.Cu" "*.Mask"))
+    (pad "GPIO4" thru_hole circle (at 17.78 10.16) (size 2 2) (drill 1) (layers "*.Cu" "*.Mask") (net 7 "BUZZER_PWM_GPIO4"))
+    (pad "GPIO3" thru_hole circle (at 17.78 12.70) (size 2 2) (drill 1) (layers "*.Cu" "*.Mask") (net 9 "ADC_BAT_GPIO3"))
+    (pad "GPIO2" thru_hole circle (at 17.78 15.24) (size 2 2) (drill 1) (layers "*.Cu" "*.Mask"))
+    (pad "GPIO1" thru_hole circle (at 17.78 17.78) (size 2 2) (drill 1) (layers "*.Cu" "*.Mask"))
+    (pad "GPIO0" thru_hole circle (at 17.78 20.32) (size 2 2) (drill 1) (layers "*.Cu" "*.Mask"))
   )
 )
